Commit message: Add schunk-mpz45 gripper support

File: schunk_mpz45/urdf/schunk_mpz45_0.xacro (robot description, xacro)
@@ -3,9 +3,3 @@
   <xacro:include filename="$(find schunk_mpz45)/urdf/schunk_mpz45_macro.xacro"/>
   <xacro:schunk_mpz45_g prefix=""/>
-  <!-- Fix robot to Gazebo world -->
-  <!-- <link name="world"/>
-  <joint name="world-base_link-fixed" type="fixed">
-    <parent link="world"/>
-    <child link="base_link"/>
-  </joint> -->
 </robot>

File: schunk_mpz45/urdf/schunk_mpz45_macro.xacro (robot description, xacro)
@@ -9,5 +9,5 @@
     <type>transmission_interface/SimpleTransmission</type>
     <joint name="${prefix}joint_7">
-      <hardwareInterface>PositionJointInterface</hardwareInterface>
+      <hardwareInterface>hardware_interface/PositionJointInterface</hardwareInterface>
     </joint>
     <actuator name="${prefix}motor7">
@@ -18,5 +18,5 @@
     <type>transmission_interface/SimpleTransmission</type>
     <joint name="${prefix}joint_8">
-      <hardwareInterface>PositionJointInterface</hardwareInterface>
+      <hardwareInterface>hardware_interface/PositionJointInterface</hardwareInterface>
     </joint>
     <actuator name="${prefix}motor8">
@@ -27,5 +27,5 @@
     <type>transmission_interface/SimpleTransmission</type>
     <joint name="${prefix}joint_9">
-      <hardwareInterface>PositionJointInterface</hardwareInterface>
+      <hardwareInterface>hardware_interface/PositionJointInterface</hardwareInterface>
     </joint>
     <actuator name="${prefix}motor9">
@@ -52,4 +52,5 @@
       <robotNamespace>/</robotNamespace>
       <robotSimType>gazebo_ros_control/DefaultRobotHWSim</robotSimType>
+      <legacyModeNS>true</legacyModeNS>
     </plugin>
   </gazebo>

File: schunk_mpz45/urdf/schunk_mpz45_macro_2.xacro (robot description, xacro)
@@ -6,9 +6,9 @@
             <inertial>
                 <mass value="1" />
-                <origin rpy="0 0 -1.57079" xyz="0 0 0" />
+                <origin rpy="0 0 -1.57079632679" xyz="0 0 0" />
                 <inertia ixx="0.001" ixy="0" ixz="0" iyy="0.001" iyz="0" izz="0.001" />
             </inertial>
             <visual>
-                <origin rpy="0 0 -1.57079" xyz="0 0 0" />
+                <origin rpy="0 0 -1.57079632679" xyz="0 0 0" />
                 <geometry>
                     <mesh filename="package://schunk_mpz45/stl/SchunkGripperNoGripperCorrect.stl" />
@@ -17,5 +17,5 @@
             </visual>
             <collision>
-                <origin rpy="0 0 -1.57079" xyz="0 0 0" />
+                <origin rpy="0 0 -1.57079632679" xyz="0 0 0" />
                 <geometry>
                     <mesh filename="package://schunk_mpz45/stl/SchunkGripperNoGripperCorrect.stl" />
@@ -29,18 +29,18 @@
             <inertial>
                 <mass value="1" />
-                <origin rpy="0 0 -1.57079" xyz="0 0 0" />
+                <origin rpy="1.57079632679 0  -1.57079632679" xyz="0 0 0" />
                 <inertia ixx="0.001" ixy="0" ixz="0" iyy="0.001" iyz="0" izz="0.001" />
             </inertial>
             <visual>
-                <origin rpy="0 0 -1.57079" xyz="0 0 0" />
+                <origin rpy="1.57079632679 0  -1.57079632679" xyz="0 0 0" />
                 <geometry>
-                    <mesh filename="package://schunk_mpz45/stl/SchunkSingleGripper1.stl" />
+                    <mesh filename="package://schunk_mpz45/stl/SchunkSingleGripper3.stl" />
                 </geometry>
-                <xacro:material_abb_black />
+                <xacro:material_abb_white />
             </visual>
             <collision>
-                <origin rpy="0 0 -1.57079" xyz="0 0 0" />
+                <origin rpy="1.57079632679 0  -1.57079632679" xyz="0 0 0" />
                 <geometry>
-                    <mesh filename="package://schunk_mpz45/stl/SchunkSingleGripper1.stl" />
+                    <mesh filename="package://schunk_mpz45/stl/SchunkSingleGripper3.stl" />
                 </geometry>
                 <material name="">
@@ -52,18 +52,18 @@
             <inertial>
                 <mass value="1" />
-                <origin rpy="0 0 -1.57079" xyz="0 0 0" />
+                <origin rpy="1.57079632679 0  -1.57079632679" xyz="0 0 0" />
                 <inertia ixx="0.001" ixy="0" ixz="0" iyy="0.001" iyz="0" izz="0.001" />
             </inertial>
             <visual>
-                <origin rpy="0 0 -1.57079" xyz="0 0 0" />
+                <origin rpy="1.57079632679 0  -1.57079632679" xyz="0 0 0" />
                 <geometry>
-                    <mesh filename="package://schunk_mpz45/stl/SchunkSingleGripper2.stl" />
+                    <mesh filename="package://schunk_mpz45/stl/SchunkSingleGripper3.stl" />
                 </geometry>
-                <xacro:material_abb_black />
+                <xacro:material_abb_white />
             </visual>
             <collision>
-                <origin rpy="0 0 -1.57079" xyz="0 0 0" />
+                <origin rpy="1.57079632679 0  -1.57079632679" xyz="0 0 0" />
                 <geometry>
-                    <mesh filename="package://schunk_mpz45/stl/SchunkSingleGripper2.stl" />
+                    <mesh filename="package://schunk_mpz45/stl/SchunkSingleGripper3.stl" />
                 </geometry>
                 <material name="">
@@ -75,16 +75,16 @@
             <inertial>
                 <mass value="1" />
-                <origin rpy="0 0 -1.57079" xyz="0 0 0" />
+                <origin rpy="1.57079632679 0  -1.57079632679" xyz="0 0 0" />
                 <inertia ixx="0.001" ixy="0" ixz="0" iyy="0.001" iyz="0" izz="0.001" />
             </inertial>
             <visual>
-                <origin rpy="0 0 -1.57079" xyz="0 0 0" />
+                <origin rpy="1.57079632679 0  -1.57079632679" xyz="0 0 0" />
                 <geometry>
                     <mesh filename="package://schunk_mpz45/stl/SchunkSingleGripper3.stl" />
                 </geometry>
-                <xacro:material_abb_black />
+                <xacro:material_abb_white />
             </visual>
             <collision>
-                <origin rpy="0 0 -1.57079" xyz="0 0 0" />
+                <origin rpy="1.57079632679 0  -1.57079632679" xyz="0 0 0" />
                 <geometry>
                     <mesh filename="package://schunk_mpz45/stl/SchunkSingleGripper3.stl" />
@@ -96,33 +96,27 @@
         </link>
         <joint name="${prefix}joint_7" type="prismatic">
-            <origin rpy="0 0 0" xyz="0 0 0" />
+            <origin rpy="-1.57079632679 -2.61799387799 -1.57079632679" xyz="0 0 0" />
             <parent link="${prefix}head" />
             <child link="${prefix}gripper1" />
-            <limit effort="0" lower="0" upper="0" velocity="0" />
+            <limit effort="0" lower="0" upper="0.005" velocity="0" />
             <axis xyz="1 0 0" />
             <dynamics damping="0.0" friction="100.0" />
         </joint>
         <joint name="${prefix}joint_8" type="prismatic">
-            <origin rpy="0 0 0" xyz="0 0 0" />
+            <origin rpy="-1.57079632679 -0.52359877559 -1.57079632679" xyz="0 0 0" />
             <parent link="${prefix}head" />
             <child link="${prefix}gripper2" />
-            <limit effort="0" lower="0" upper="0" velocity="0" />
+            <limit effort="0" lower="0" upper="0.005" velocity="0" />
             <axis xyz="1 0 0" />
+            <mimic joint="${prefix}joint_7" multiplier="1" offset="0"/>
             <dynamics damping="0.0" friction="100.0" />
         </joint>
         <joint name="${prefix}joint_9" type="prismatic">
-            <origin rpy="0 0 0" xyz="0 0 0" />
+            <origin rpy="0 1.57079632679632679 0" xyz="0 0 0" />
             <parent link="${prefix}head" />
             <child link="${prefix}gripper3" />
-            <limit effort="0" lower="0" upper="0" velocity="0" />
+            <limit effort="0" lower="0" upper="0.005" velocity="0" />
             <axis xyz="1 0 0" />
-            <dynamics damping="0.0" friction="100.0" />
-        </joint>
-        <joint name="${prefix}joint_10" type="fixed">
-            <origin rpy="0 0 0" xyz="0 0 0" />
-            <parent link="${prefix}tool0" />
-            <child link="${prefix}head" />
-            <limit effort="0" lower="0" upper="0" velocity="0" />
-            <axis xyz="1 0 0" />
+            <mimic joint="${prefix}joint_7" multiplier="1" offset="0"/>
             <dynamics damping="0.0" friction="100.0" />
         </joint>

File: simulation/urdf/abb_irb120_schunk_mpz45.xacro (robot description, xacro)
@@ -3,7 +3,20 @@
     <xacro:include filename="$(find abb_irb120_gazebo)/urdf/irb120_3_58.xacro" />
     <xacro:include filename="$(find schunk_mpz45)/urdf/schunk_mpz45_0.xacro" />
+    <joint name="joint_10" type="fixed">
+        <origin rpy="0 0 0" xyz="0 0 0" />
+        <parent link="tool0" />
+        <child link="head" />
+        <limit effort="0" lower="0" upper="0" velocity="0" />
+        <axis xyz="1 0 0" />
+        <dynamics damping="0.0" friction="100.0" />
+    </joint>
     <xacro:macro name="abb_irb120_schunk_mpz45" params="">
         <xacro:abb_irb120_3_58 prefix="" />
         <xacro:schunk_mpz45 prefix="" />
+        <link name="world" />
+        <joint name="world-base_link-fixed" type="fixed">
+            <parent link="world" />
+            <child link="base_link" />
+        </joint>
     </xacro:macro>
 </robot>
