Commit message: Add kinematics for the ABB-IRB120 + Schunk mpz45

File: schunk_mpz45/urdf/schunk_mpz45_macro_2.xacro (robot description, xacro)
@@ -95,4 +95,15 @@
             </collision>
         </link>
+        <link name="${prefix}eef">
+            <visual>
+                <origin xyz="0 0 0" rpy="0 0 0" />
+                <geometry>
+                    <sphere radius="0.001"/>
+                </geometry>
+                <material name="Cyan">
+                  <color rgba="0 1.0 1.0 1.0"/>
+                </material>
+              </visual>
+        </link>
         <joint name="${prefix}joint_7" type="prismatic">
             <origin rpy="${-1 / 2 * pi} ${-5 / 6 * pi} ${-1 / 2 * pi}" xyz="0 0 0" />
@@ -115,4 +126,9 @@
             <mimic joint="${prefix}joint_7"/>
         </joint>
+        <joint name="${prefix}eef-head" type="fixed">
+            <origin rpy="0 0 0" xyz="0.05 0 0" />
+            <parent link="${prefix}head" />
+            <child link="${prefix}eef" />
+        </joint>
     </xacro:macro>
 </robot>
