Commit message: Minor changes in Appereance Add correct specifications of Schunk mpz45

File: abb_irb120_gazebo/urdf/irb120_3_58_macro.xacro (robot description, xacro)
@@ -9,5 +9,5 @@
     <type>transmission_interface/SimpleTransmission</type>
     <joint name="${prefix}joint_1">
-      <hardwareInterface>PositionJointInterface</hardwareInterface>
+      <hardwareInterface>hardware_interface/PositionJointInterface</hardwareInterface>
     </joint>
     <actuator name="${prefix}motor1">
@@ -18,5 +18,5 @@
     <type>transmission_interface/SimpleTransmission</type>
     <joint name="${prefix}joint_2">
-      <hardwareInterface>PositionJointInterface</hardwareInterface>
+      <hardwareInterface>hardware_interface/PositionJointInterface</hardwareInterface>
     </joint>
     <actuator name="${prefix}motor2">
@@ -27,5 +27,5 @@
     <type>transmission_interface/SimpleTransmission</type>
     <joint name="${prefix}joint_3">
-      <hardwareInterface>PositionJointInterface</hardwareInterface>
+      <hardwareInterface>hardware_interface/PositionJointInterface</hardwareInterface>
     </joint>
     <actuator name="${prefix}motor3">
@@ -36,5 +36,5 @@
     <type>transmission_interface/SimpleTransmission</type>
     <joint name="${prefix}joint_4">
-      <hardwareInterface>PositionJointInterface</hardwareInterface>
+      <hardwareInterface>hardware_interface/PositionJointInterface</hardwareInterface>
     </joint>
     <actuator name="${prefix}motor4">
@@ -45,5 +45,5 @@
     <type>transmission_interface/SimpleTransmission</type>
     <joint name="${prefix}joint_5">
-      <hardwareInterface>PositionJointInterface</hardwareInterface>
+      <hardwareInterface>hardware_interface/PositionJointInterface</hardwareInterface>
     </joint>
     <actuator name="${prefix}motor5">
@@ -54,5 +54,5 @@
     <type>transmission_interface/SimpleTransmission</type>
     <joint name="${prefix}joint_6">
-      <hardwareInterface>PositionJointInterface</hardwareInterface>
+      <hardwareInterface>hardware_interface/PositionJointInterface</hardwareInterface>
     </joint>
     <actuator name="${prefix}motor6">
@@ -95,4 +95,5 @@
       <robotNamespace>/</robotNamespace>
       <robotSimType>gazebo_ros_control/DefaultRobotHWSim</robotSimType>
+      <legacyModeNS>true</legacyModeNS>
     </plugin>
   </gazebo>

File: abb_irb120_gazebo/urdf/irb120t_3_58_macro.xacro (robot description, xacro)
@@ -9,5 +9,5 @@
     <type>transmission_interface/SimpleTransmission</type>
     <joint name="${prefix}joint_1">
-      <hardwareInterface>PositionJointInterface</hardwareInterface>
+      <hardwareInterface>hardware_interface/PositionJointInterface</hardwareInterface>
     </joint>
     <actuator name="${prefix}motor1">
@@ -18,5 +18,5 @@
     <type>transmission_interface/SimpleTransmission</type>
     <joint name="${prefix}joint_2">
-      <hardwareInterface>PositionJointInterface</hardwareInterface>
+      <hardwareInterface>hardware_interface/PositionJointInterface</hardwareInterface>
     </joint>
     <actuator name="${prefix}motor2">
@@ -27,5 +27,5 @@
     <type>transmission_interface/SimpleTransmission</type>
     <joint name="${prefix}joint_3">
-      <hardwareInterface>PositionJointInterface</hardwareInterface>
+      <hardwareInterface>hardware_interface/PositionJointInterface</hardwareInterface>
     </joint>
     <actuator name="${prefix}motor3">
@@ -36,5 +36,5 @@
     <type>transmission_interface/SimpleTransmission</type>
     <joint name="${prefix}joint_4">
-      <hardwareInterface>PositionJointInterface</hardwareInterface>
+      <hardwareInterface>hardware_interface/PositionJointInterface</hardwareInterface>
     </joint>
     <actuator name="${prefix}motor4">
@@ -45,5 +45,5 @@
     <type>transmission_interface/SimpleTransmission</type>
     <joint name="${prefix}joint_5">
-      <hardwareInterface>PositionJointInterface</hardwareInterface>
+      <hardwareInterface>hardware_interface/PositionJointInterface</hardwareInterface>
     </joint>
     <actuator name="${prefix}motor5">
@@ -54,5 +54,5 @@
     <type>transmission_interface/SimpleTransmission</type>
     <joint name="${prefix}joint_6">
-      <hardwareInterface>PositionJointInterface</hardwareInterface>
+      <hardwareInterface>hardware_interface/PositionJointInterface</hardwareInterface>
     </joint>
     <actuator name="${prefix}motor6">

File: schunk_mpz45/urdf/schunk_mpz45_macro.xacro (robot description, xacro)
@@ -35,14 +35,18 @@
   <!-- end of transmission list -->
   <!-- Gazebo-specific link properties -->
-  <gazebo reference="${prefix}link_7">
-    <material>Gazebo/Black</material>
+  <gazebo reference="${prefix}head">
+    <material>Gazebo/Grey</material>
     <turnGravityOff>true</turnGravityOff>
   </gazebo>
-  <gazebo reference="${prefix}link_8">
-    <material>Gazebo/Black</material>
+  <gazebo reference="${prefix}gripper1">
+    <material>Gazebo/White</material>
     <turnGravityOff>true</turnGravityOff>
   </gazebo>
-  <gazebo reference="${prefix}link_9">
-    <material>Gazebo/Black</material>
+  <gazebo reference="${prefix}gripper2">
+    <material>Gazebo/White</material>
+    <turnGravityOff>true</turnGravityOff>
+  </gazebo>
+  <gazebo reference="${prefix}gripper3">
+    <material>Gazebo/White</material>
     <turnGravityOff>true</turnGravityOff>
   </gazebo>

File: schunk_mpz45/urdf/schunk_mpz45_macro_2.xacro (robot description, xacro)
@@ -6,9 +6,9 @@
             <inertial>
                 <mass value="1" />
-                <origin rpy="0 0 -1.57079632679" xyz="0 0 0" />
+                <origin rpy="0 0 ${-1 / 2 * pi}" xyz="0 0 0" />
                 <inertia ixx="0.001" ixy="0" ixz="0" iyy="0.001" iyz="0" izz="0.001" />
             </inertial>
             <visual>
-                <origin rpy="0 0 -1.57079632679" xyz="0 0 0" />
+                <origin rpy="0 0 ${-1 / 2 * pi}" xyz="0 0 0" />
                 <geometry>
                     <mesh filename="package://schunk_mpz45/stl/SchunkGripperNoGripperCorrect.stl" />
@@ -17,5 +17,5 @@
             </visual>
             <collision>
-                <origin rpy="0 0 -1.57079632679" xyz="0 0 0" />
+                <origin rpy="0 0 ${-1 / 2 * pi}" xyz="0 0 0" />
                 <geometry>
                     <mesh filename="package://schunk_mpz45/stl/SchunkGripperNoGripperCorrect.stl" />
@@ -29,9 +29,9 @@
             <inertial>
                 <mass value="1" />
-                <origin rpy="1.57079632679 0  -1.57079632679" xyz="0 0 0" />
+                <origin rpy="${1 / 2 * pi} 0  ${-1 / 2 * pi}" xyz="0 0 0" />
                 <inertia ixx="0.001" ixy="0" ixz="0" iyy="0.001" iyz="0" izz="0.001" />
             </inertial>
             <visual>
-                <origin rpy="1.57079632679 0  -1.57079632679" xyz="0 0 0" />
+                <origin rpy="${1 / 2 * pi} 0  ${-1 / 2 * pi}" xyz="0 0 0" />
                 <geometry>
                     <mesh filename="package://schunk_mpz45/stl/SchunkSingleGripper3.stl" />
@@ -40,5 +40,5 @@
             </visual>
             <collision>
-                <origin rpy="1.57079632679 0  -1.57079632679" xyz="0 0 0" />
+                <origin rpy="${1 / 2 * pi} 0  ${-1 / 2 * pi}" xyz="0 0 0" />
                 <geometry>
                     <mesh filename="package://schunk_mpz45/stl/SchunkSingleGripper3.stl" />
@@ -52,9 +52,9 @@
             <inertial>
                 <mass value="1" />
-                <origin rpy="1.57079632679 0  -1.57079632679" xyz="0 0 0" />
+                <origin rpy="${1 / 2 * pi} 0  ${-1 / 2 * pi}" xyz="0 0 0" />
                 <inertia ixx="0.001" ixy="0" ixz="0" iyy="0.001" iyz="0" izz="0.001" />
             </inertial>
             <visual>
-                <origin rpy="1.57079632679 0  -1.57079632679" xyz="0 0 0" />
+                <origin rpy="${1 / 2 * pi} 0  ${-1 / 2 * pi}" xyz="0 0 0" />
                 <geometry>
                     <mesh filename="package://schunk_mpz45/stl/SchunkSingleGripper3.stl" />
@@ -63,5 +63,5 @@
             </visual>
             <collision>
-                <origin rpy="1.57079632679 0  -1.57079632679" xyz="0 0 0" />
+                <origin rpy="${1 / 2 * pi} 0  ${-1 / 2 * pi}" xyz="0 0 0" />
                 <geometry>
                     <mesh filename="package://schunk_mpz45/stl/SchunkSingleGripper3.stl" />
@@ -75,9 +75,9 @@
             <inertial>
                 <mass value="1" />
-                <origin rpy="1.57079632679 0  -1.57079632679" xyz="0 0 0" />
+                <origin rpy="${1 / 2 * pi} 0  ${-1 / 2 * pi}" xyz="0 0 0" />
                 <inertia ixx="0.001" ixy="0" ixz="0" iyy="0.001" iyz="0" izz="0.001" />
             </inertial>
             <visual>
-                <origin rpy="1.57079632679 0  -1.57079632679" xyz="0 0 0" />
+                <origin rpy="${1 / 2 * pi} 0  ${-1 / 2 * pi}" xyz="0 0 0" />
                 <geometry>
                     <mesh filename="package://schunk_mpz45/stl/SchunkSingleGripper3.stl" />
@@ -86,5 +86,5 @@
             </visual>
             <collision>
-                <origin rpy="1.57079632679 0  -1.57079632679" xyz="0 0 0" />
+                <origin rpy="${1 / 2 * pi} 0  ${-1 / 2 * pi}" xyz="0 0 0" />
                 <geometry>
                     <mesh filename="package://schunk_mpz45/stl/SchunkSingleGripper3.stl" />
@@ -96,29 +96,24 @@
         </link>
         <joint name="${prefix}joint_7" type="prismatic">
-            <origin rpy="-1.57079632679 -2.61799387799 -1.57079632679" xyz="0 0 0" />
+            <origin rpy="${-1 / 2 * pi} ${-5 / 6 * pi} ${-1 / 2 * pi}" xyz="0 0 0" />
             <parent link="${prefix}head" />
             <child link="${prefix}gripper1" />
-            <limit effort="0" lower="0" upper="0.005" velocity="0" />
-            <axis xyz="1 0 0" />
-            <dynamics damping="0.0" friction="100.0" />
+            <limit effort="310" lower="0" upper="0.005" velocity="0.1"/>
         </joint>
         <joint name="${prefix}joint_8" type="prismatic">
-            <origin rpy="-1.57079632679 -0.52359877559 -1.57079632679" xyz="0 0 0" />
+            <origin rpy="${-1 / 2 * pi} ${-1 / 6 * pi} ${-1 / 2 * pi}" xyz="0 0 0" />
             <parent link="${prefix}head" />
             <child link="${prefix}gripper2" />
-            <limit effort="0" lower="0" upper="0.005" velocity="0" />
-            <axis xyz="1 0 0" />
-            <mimic joint="${prefix}joint_7" multiplier="1" offset="0"/>
-            <dynamics damping="0.0" friction="100.0" />
+            <limit effort="310" lower="0" upper="0.005" velocity="0.1" />
+            <mimic joint="${prefix}joint_7"/>
         </joint>
         <joint name="${prefix}joint_9" type="prismatic">
-            <origin rpy="0 1.57079632679632679 0" xyz="0 0 0" />
+            <origin rpy="0 ${1 / 2 * pi} 0" xyz="0 0 0" />
             <parent link="${prefix}head" />
             <child link="${prefix}gripper3" />
-            <limit effort="0" lower="0" upper="0.005" velocity="0" />
-            <axis xyz="1 0 0" />
-            <mimic joint="${prefix}joint_7" multiplier="1" offset="0"/>
-            <dynamics damping="0.0" friction="100.0" />
+            <limit effort="310" lower="0" upper="0.005" velocity="0.1" />
+            <mimic joint="${prefix}joint_7"/>
         </joint>
     </xacro:macro>
 </robot>
+<!-- Schunk specifications according to:  https://schunk.com/fileadmin/pim/docs/IM0020092.PDF-->

File: simulation/urdf/abb_irb120_schunk_mpz45.xacro (robot description, xacro)
@@ -2,12 +2,9 @@
 <robot name="abb_irb120_3_58_schunk" xmlns:xacro="http://ros.org/wiki/xacro">
     <xacro:include filename="$(find abb_irb120_gazebo)/urdf/irb120_3_58.xacro" />
-    <xacro:include filename="$(find schunk_mpz45)/urdf/schunk_mpz45_0.xacro" />
+    <xacro:include filename="$(find schunk_mpz45)/urdf/schunk_mpz45.xacro" />
     <joint name="joint_10" type="fixed">
         <origin rpy="0 0 0" xyz="0 0 0" />
         <parent link="tool0" />
         <child link="head" />
-        <limit effort="0" lower="0" upper="0" velocity="0" />
-        <axis xyz="1 0 0" />
-        <dynamics damping="0.0" friction="100.0" />
     </joint>
     <xacro:macro name="abb_irb120_schunk_mpz45" params="">
