Commit message: Fixed robotarm movement with gripper

File: abb_irb120_gazebo/urdf/irb120_3_58.xacro (robot description, xacro)
@@ -1,6 +1,347 @@
-<?xml version="1.0" ?>
-<robot name="abb_irb120_3_58" xmlns:xacro="http://ros.org/wiki/xacro">
-  <xacro:include filename="$(find abb_irb120_gazebo)/urdf/irb120_3_58_macro.xacro"/>
-  <xacro:abb_irb120_3_58_g prefix=""/>
+<?xml version="1.0" encoding="utf-8"?>
+<!-- =================================================================================== -->
+<!-- |    This document was autogenerated by xacro from abb_irb120_schunk_mpz45.xacro  | -->
+<!-- |    EDITING THIS FILE BY HAND IS NOT RECOMMENDED                                 | -->
+<!-- =================================================================================== -->
+<!-- =================================================================================== -->
+<!-- |    This document was autogenerated by xacro from abb_irb120_schunk_mpz45.xacro  | -->
+<!-- |    EDITING THIS FILE BY HAND IS NOT RECOMMENDED                                 | -->
+<!-- =================================================================================== -->
+<robot name="abb_irb120_schunk_mpz45">
+  <!-- Conversion were obtained from http://www.e-paint.co.uk/Lab_values.asp
+       unless otherwise stated. -->
+  <!-- link list -->
+  <link name="base_link">
+    <inertial>
+      <mass value="6.215"/>
+      <origin rpy="0 0 0" xyz="-0.04204 8.01E-05 0.07964"/>
+      <inertia ixx="0.0247272" ixy="-8.0784E-05" ixz="0.00130902" iyy="0.0491285" iyz="-8.0419E-06" izz="0.0472376"/>
+    </inertial>
+    <visual>
+      <origin rpy="0 0 0" xyz="0 0 0"/>
+      <geometry>
+        <mesh filename="package://abb_irb120_support/meshes/irb120_3_58/visual/base_link.stl"/>
+      </geometry>
+      <material name="">
+        <color rgba="0.7372549 0.3490196 0.1607843 1"/>
+      </material>
+    </visual>
+    <collision>
+      <origin rpy="0 0 0" xyz="0 0 0"/>
+      <geometry>
+        <mesh filename="package://abb_irb120_support/meshes/irb120_3_58/collision/base_link.stl"/>
+      </geometry>
+      <material name="">
+        <color rgba="1 1 0 1"/>
+      </material>
+    </collision>
+  </link>
+  <link name="link_1">
+    <inertial>
+      <mass value="3.067"/>
+      <origin rpy="0 0 0" xyz="9.77E-05 -0.00012 0.23841"/>
+      <inertia ixx="0.0142175" ixy="-1.28579E-05" ixz="-2.31364E-05" iyy="0.0144041" iyz="1.93404E-05" izz="0.0104533"/>
+    </inertial>
+    <visual>
+      <origin rpy="0 0 0" xyz="0 0 0"/>
+      <geometry>
+        <mesh filename="package://abb_irb120_support/meshes/irb120_3_58/visual/link_1.stl"/>
+      </geometry>
+      <material name="">
+        <color rgba="0.7372549 0.3490196 0.1607843 1"/>
+      </material>
+    </visual>
+    <collision>
+      <origin rpy="0 0 0" xyz="0 0 0"/>
+      <geometry>
+        <mesh filename="package://abb_irb120_support/meshes/irb120_3_58/collision/link_1.stl"/>
+      </geometry>
+      <material name="">
+        <color rgba="1 1 0 1"/>
+      </material>
+    </collision>
+  </link>
+  <link name="link_2">
+    <inertial>
+      <mass value="3.909"/>
+      <origin rpy="0 0 0" xyz="0.00078 -0.00212 0.10124"/>
+      <inertia ixx="0.0603111" ixy="9.83431E-06" ixz="5.72407E-05" iyy="0.041569" iyz="-0.00050497" izz="0.0259548"/>
+    </inertial>
+    <visual>
+      <origin rpy="0 0 0" xyz="0 0 0"/>
+      <geometry>
+        <mesh filename="package://abb_irb120_support/meshes/irb120_3_58/visual/link_2.stl"/>
+      </geometry>
+      <material name="">
+        <color rgba="0.7372549 0.3490196 0.1607843 1"/>
+      </material>
+    </visual>
+    <collision>
+      <origin rpy="0 0 0" xyz="0 0 0"/>
+      <geometry>
+        <mesh filename="package://abb_irb120_support/meshes/irb120_3_58/collision/link_2.stl"/>
+      </geometry>
+      <material name="">
+        <color rgba="1 1 0 1"/>
+      </material>
+    </collision>
+  </link>
+  <link name="link_3">
+    <inertial>
+      <mass value="2.944"/>
+      <origin rpy="0 0 0" xyz="0.02281 0.00106 0.05791"/>
+      <inertia ixx="0.00835606" ixy="-8.01545E-05" ixz="0.00142884" iyy="0.016713" iyz="-0.000182227" izz="0.0126984"/>
+    </inertial>
+    <visual>
+      <origin rpy="0 0 0" xyz="0 0 0"/>
+      <geometry>
+        <mesh filename="package://abb_irb120_support/meshes/irb120_3_58/visual/link_3.stl"/>
+      </geometry>
+      <material name="">
+        <color rgba="0.7372549 0.3490196 0.1607843 1"/>
+      </material>
+    </visual>
+    <collision>
+      <origin rpy="0 0 0" xyz="0 0 0"/>
+      <geometry>
+        <mesh filename="package://abb_irb120_support/meshes/irb120_3_58/collision/link_3.stl"/>
+      </geometry>
+      <material name="">
+        <color rgba="1 1 0 1"/>
+      </material>
+    </collision>
+  </link>
+  <link name="link_4">
+    <inertial>
+      <mass value="1.328"/>
+      <origin rpy="0 0 0" xyz="0.2247 0.00015 0.00041"/>
+      <inertia ixx="0.00284661" ixy="-2.12765E-05" ixz="-1.6435E-05" iyy="0.00401346" iyz="1.31336E-05" izz="0.0052535"/>
+    </inertial>
+    <visual>
+      <origin rpy="0 0 0" xyz="0 0 0"/>
+      <geometry>
+        <mesh filename="package://abb_irb120_support/meshes/irb120_3_58/visual/link_4.stl"/>
+      </geometry>
+      <material name="">
+        <color rgba="0.7372549 0.3490196 0.1607843 1"/>
+      </material>
+    </visual>
+    <collision>
+      <origin rpy="0 0 0" xyz="0 0 0"/>
+      <geometry>
+        <mesh filename="package://abb_irb120_support/meshes/irb120_3_58/collision/link_4.stl"/>
+      </geometry>
+      <material name="">
+        <color rgba="1 1 0 1"/>
+      </material>
+    </collision>
+  </link>
+  <link name="link_5">
+    <inertial>
+      <mass value="0.546"/>
+      <origin rpy="0 0 0" xyz="-0.00109 3.68E-05 6.22E-05"/>
+      <inertia ixx="0.000404891" ixy="1.61943E-06" ixz="8.46805E-07" iyy="0.000892825" iyz="-1.51792E-08" izz="0.000815468"/>
+    </inertial>
+    <visual>
+      <origin rpy="0 0 0" xyz="0 0 0"/>
+      <geometry>
+        <mesh filename="package://abb_irb120_support/meshes/irb120_3_58/visual/link_5.stl"/>
+      </geometry>
+      <material name="">
+        <color rgba="0.7372549 0.3490196 0.1607843 1"/>
+      </material>
+    </visual>
+    <collision>
+      <origin rpy="0 0 0" xyz="0 0 0"/>
+      <geometry>
+        <mesh filename="package://abb_irb120_support/meshes/irb120_3_58/collision/link_5.stl"/>
+      </geometry>
+      <material name="">
+        <color rgba="1 1 0 1"/>
+      </material>
+    </collision>
+  </link>
+  <link name="link_6">
+    <inertial>
+      <mass value="0.137"/>
+      <origin rpy="0 0 0" xyz="-0.00706 -0.00017 -1.32E-06"/>
+      <inertia ixx="0.001" ixy="0" ixz="0" iyy="0.001" iyz="0" izz="0.001"/>
+    </inertial>
+    <visual>
+      <origin rpy="0 0 0" xyz="0 0 0"/>
+      <geometry>
+        <mesh filename="package://abb_irb120_support/meshes/irb120_3_58/visual/link_6.stl"/>
+      </geometry>
+      <material name="">
+        <color rgba="0.1882353 0.1960784 0.2039216 1"/>
+      </material>
+    </visual>
+    <collision>
+      <origin rpy="0 0 0" xyz="0 0 0"/>
+      <geometry>
+        <mesh filename="package://abb_irb120_support/meshes/irb120_3_58/collision/link_6.stl"/>
+      </geometry>
+      <material name="">
+        <color rgba="1 1 0 1"/>
+      </material>
+    </collision>
+  </link>
+  <link name="tool0"/>
+  <!-- end of link list -->
+  <!-- joint list -->
+  <joint name="joint_1" type="revolute">
+    <origin rpy="0 0 0" xyz="0 0 0"/>
+    <parent link="base_link"/>
+    <child link="link_1"/>
+    <limit effort="0" lower="-2.87979" upper="2.87979" velocity="4.36332"/>
+    <axis xyz="0 0 1"/>
+    <dynamics damping="0.0" friction="0.0"/>
+  </joint>
+  <joint name="joint_2" type="revolute">
+    <origin rpy="0 0 0" xyz="0 0 0.29"/>
+    <parent link="link_1"/>
+    <child link="link_2"/>
+    <limit effort="0" lower="-1.91986" upper="1.91986" velocity="4.36332"/>
+    <axis xyz="0 1 0"/>
+    <dynamics damping="0.0" friction="0.0"/>
+  </joint>
+  <joint name="joint_3" type="revolute">
+    <origin rpy="0 0 0" xyz="0 0 0.27"/>
+    <parent link="link_2"/>
+    <child link="link_3"/>
+    <limit effort="0" lower="-1.91986" upper="1.22173" velocity="4.36332"/>
+    <axis xyz="0 1 0"/>
+    <dynamics damping="0.0" friction="0.0"/>
+  </joint>
+  <joint name="joint_4" type="revolute">
+    <origin rpy="0 0 0" xyz="0 0 0.07"/>
+    <parent link="link_3"/>
+    <child link="link_4"/>
+    <limit effort="0" lower="-2.79253" upper="2.79253" velocity="5.58505"/>
+    <axis xyz="1 0 0"/>
+    <dynamics damping="0.0" friction="0.0"/>
+  </joint>
+  <joint name="joint_5" type="revolute">
+    <origin rpy="0 0 0" xyz="0.302 0 0"/>
+    <parent link="link_4"/>
+    <child link="link_5"/>
+    <limit effort="0" lower="-2.094395" upper="2.094395" velocity="5.58505"/>
+    <axis xyz="0 1 0"/>
+    <dynamics damping="0.0" friction="0.0"/>
+  </joint>
+  <joint name="joint_6" type="revolute">
+    <origin rpy="0 0 0" xyz="0.072 0 0"/>
+    <parent link="link_5"/>
+    <child link="link_6"/>
+    <limit effort="0" lower="-6.98132" upper="6.98132" velocity="7.33038"/>
+    <axis xyz="1 0 0"/>
+    <dynamics damping="0.0" friction="0.0"/>
+  </joint>
+  <joint name="joint6-tool0" type="fixed">
+    <parent link="link_6"/>
+    <child link="tool0"/>
+    <origin rpy="0 0 0" xyz="0 0 0"/>
+  </joint>
+  <!-- end of joint list -->
+  <!-- ROS base_link to ABB World Coordinates transform -->
+  <link name="base"/>
+  <joint name="base_link-base" type="fixed">
+    <origin rpy="0 0 0" xyz="0 0 0"/>
+    <parent link="base_link"/>
+    <child link="base"/>
+  </joint>
+  <!-- transmission list -->
+  <transmission name="tran1">
+    <type>transmission_interface/SimpleTransmission</type>
+    <joint name="joint_1">
+      <hardwareInterface>hardware_interface/PositionJointInterface</hardwareInterface>
+    </joint>
+    <actuator name="motor1">
+      <mechanicalReduction>1</mechanicalReduction>
+    </actuator>
+  </transmission>
+  <transmission name="tran2">
+    <type>transmission_interface/SimpleTransmission</type>
+    <joint name="joint_2">
+      <hardwareInterface>hardware_interface/PositionJointInterface</hardwareInterface>
+    </joint>
+    <actuator name="motor2">
+      <mechanicalReduction>1</mechanicalReduction>
+    </actuator>
+  </transmission>
+  <transmission name="tran3">
+    <type>transmission_interface/SimpleTransmission</type>
+    <joint name="joint_3">
+      <hardwareInterface>hardware_interface/PositionJointInterface</hardwareInterface>
+    </joint>
+    <actuator name="motor3">
+      <mechanicalReduction>1</mechanicalReduction>
+    </actuator>
+  </transmission>
+  <transmission name="tran4">
+    <type>transmission_interface/SimpleTransmission</type>
+    <joint name="joint_4">
+      <hardwareInterface>hardware_interface/PositionJointInterface</hardwareInterface>
+    </joint>
+    <actuator name="motor4">
+      <mechanicalReduction>1</mechanicalReduction>
+    </actuator>
+  </transmission>
+  <transmission name="tran5">
+    <type>transmission_interface/SimpleTransmission</type>
+    <joint name="joint_5">
+      <hardwareInterface>hardware_interface/PositionJointInterface</hardwareInterface>
+    </joint>
+    <actuator name="motor5">
+      <mechanicalReduction>1</mechanicalReduction>
+    </actuator>
+  </transmission>
+  <transmission name="tran6">
+    <type>transmission_interface/SimpleTransmission</type>
+    <joint name="joint_6">
+      <hardwareInterface>hardware_interface/PositionJointInterface</hardwareInterface>
+    </joint>
+    <actuator name="motor6">
+      <mechanicalReduction>1</mechanicalReduction>
+    </actuator>
+  </transmission>
+  <!-- end of transmission list -->
+  <!-- Gazebo-specific link properties -->
+  <gazebo reference="base_link">
+    <material>Gazebo/Orange</material>
+    <turnGravityOff>true</turnGravityOff>
+  </gazebo>
+  <gazebo reference="link_1">
+    <material>Gazebo/Orange</material>
+    <turnGravityOff>true</turnGravityOff>
+  </gazebo>
+  <gazebo reference="link_2">
+    <material>Gazebo/Orange</material>
+    <turnGravityOff>true</turnGravityOff>
+  </gazebo>
+  <gazebo reference="link_3">
+    <material>Gazebo/Orange</material>
+    <turnGravityOff>true</turnGravityOff>
+  </gazebo>
+  <gazebo reference="link_4">
+    <material>Gazebo/Orange</material>
+    <turnGravityOff>true</turnGravityOff>
+  </gazebo>
+  <gazebo reference="link_5">
+    <material>Gazebo/Orange</material>
+    <turnGravityOff>true</turnGravityOff>
+  </gazebo>
+  <gazebo reference="link_6">
+    <material>Gazebo/Black</material>
+    <turnGravityOff>true</turnGravityOff>
+  </gazebo>
+  <!-- ros_control plugin -->
+  <gazebo>
+    <plugin filename="libgazebo_ros_control.so" name="gazebo_ros_control">
+      <robotNamespace>/</robotNamespace>
+      <robotSimType>gazebo_ros_control/DefaultRobotHWSim</robotSimType>
+      <legacyModeNS>true</legacyModeNS>
+    </plugin>
+  </gazebo>
   <!-- Fix robot to Gazebo world -->
   <link name="world"/>
@@ -9,3 +350,193 @@
     <child link="base_link"/>
   </joint>
+  <!-- Conversion were obtained from http://www.e-paint.co.uk/Lab_values.asp
+       unless otherwise stated. -->
+  <link name="head">
+    <inertial>
+      <mass value="1"/>
+      <origin rpy="0 0 -1.57079632679" xyz="0 0 0"/>
+      <inertia ixx="0.001" ixy="0" ixz="0" iyy="0.001" iyz="0" izz="0.001"/>
+    </inertial>
+    <visual>
+      <origin rpy="0 0 -1.57079632679" xyz="0 0 0"/>
+      <geometry>
+        <mesh filename="package://schunk_mpz45/stl/SchunkGripperNoGripperCorrect.stl"/>
+      </geometry>
+      <material name="">
+        <color rgba="0.1882353 0.1960784 0.2039216 1"/>
+      </material>
+    </visual>
+    <collision>
+      <origin rpy="0 0 -1.57079632679" xyz="0 0 0"/>
+      <geometry>
+        <mesh filename="package://schunk_mpz45/stl/SchunkGripperNoGripperCorrect.stl"/>
+      </geometry>
+      <material name="">
+        <color rgba="1 1 0 1"/>
+      </material>
+    </collision>
+  </link>
+  <link name="gripper1">
+    <inertial>
+      <mass value="1"/>
+      <origin rpy="1.57079632679 0  -1.57079632679" xyz="0 0 0"/>
+      <inertia ixx="0.001" ixy="0" ixz="0" iyy="0.001" iyz="0" izz="0.001"/>
+    </inertial>
+    <visual>
+      <origin rpy="1.57079632679 0  -1.57079632679" xyz="0 0 0"/>
+      <geometry>
+        <mesh filename="package://schunk_mpz45/stl/SchunkSingleGripper3.stl"/>
+      </geometry>
+      <material name="">
+        <color rgba="0.9254902 0.9254902 0.9058824 1"/>
+      </material>
+    </visual>
+    <collision>
+      <origin rpy="1.57079632679 0  -1.57079632679" xyz="0 0 0"/>
+      <geometry>
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
File: pickuppoint/urdf/pickuppoint.xacro (robot description, xacro)
@@ -15,5 +15,5 @@
             <origin rpy="0 0 0" xyz="0.00 0.395 0" />
             <geometry>
-                <mesh filename="package://pickuppoint/stl/ultimateLowResPickupPoint2.0.stl" />
+                <mesh filename="package://pickuppoint/stl/PickupPoint.stl" />
             </geometry>
             <material name="red">
@@ -24,5 +24,5 @@
             <origin rpy="0 0 0" xyz="0.0 0.395 0" />
             <geometry>
-                <mesh filename="package://pickuppoint/stl/ultimateLowResPickupPoint2.0.stl" />
+                <mesh filename="package://pickuppoint/stl/ultimateLowResPickupPoint3.0.stl" />
             </geometry>
             <material name="">

Commit message: Implemented gripper control from ros-action

File: abb_irb120_gazebo/urdf/irb120_3_58.xacro (robot description, xacro)
@@ -492,7 +492,8 @@
     <type>transmission_interface/SimpleTransmission</type>
     <joint name="joint_7">
-      <hardwareInterface>hardware_interface/PositionJointInterface</hardwareInterface>
+      <hardwareInterface>hardware_interface/EffortJointInterface</hardwareInterface>
     </joint>
     <actuator name="motor7">
+      <hardwareInterface>hardware_interface/EffortJointInterface</hardwareInterface>
       <mechanicalReduction>1</mechanicalReduction>
     </actuator>
@@ -501,7 +502,8 @@
     <type>transmission_interface/SimpleTransmission</type>
     <joint name="joint_8">
-      <hardwareInterface>hardware_interface/PositionJointInterface</hardwareInterface>
+      <hardwareInterface>hardware_interface/EffortJointInterface</hardwareInterface>
     </joint>
     <actuator name="motor8">
+      <hardwareInterface>hardware_interface/EffortJointInterface</hardwareInterface>
       <mechanicalReduction>1</mechanicalReduction>
     </actuator>
@@ -510,7 +512,8 @@
     <type>transmission_interface/SimpleTransmission</type>
     <joint name="joint_9">
-      <hardwareInterface>hardware_interface/PositionJointInterface</hardwareInterface>
+      <hardwareInterface>hardware_interface/EffortJointInterface</hardwareInterface>
     </joint>
     <actuator name="motor9">
+      <hardwareInterface>hardware_interface/EffortJointInterface</hardwareInterface>
       <mechanicalReduction>1</mechanicalReduction>
     </actuator>

File: schunk_mpz45/urdf/schunk_mpz45_macro.xacro (robot description, xacro)
@@ -54,5 +54,5 @@
   <gazebo>
     <plugin name="gazebo_ros_control" filename="libgazebo_ros_control.so">
-      <robotNamespace>/</robotNamespace>
+      <robotNamespace>/simple_model</robotNamespace>
       <robotSimType>gazebo_ros_control/DefaultRobotHWSim</robotSimType>
       <legacyModeNS>true</legacyModeNS>

File: schunk_mpz45/urdf/schunk_mpz45_macro_2.xacro (robot description, xacro)
@@ -102,7 +102,7 @@
                 </geometry>
                 <material name="Cyan">
-                  <color rgba="0 1.0 1.0 1.0"/>
+                    <color rgba="0 1.0 1.0 1.0"/>
                 </material>
-              </visual>
+            </visual>
         </link>
         <joint name="${prefix}joint_7" type="prismatic">

Commit message: Add TF2 Support for robot movements Movements can now be made regardless of the position of the robot or any objects it needs to move to.

File: abb_irb120_gazebo/urdf/irb120_3_58.xacro (robot description, xacro)
@@ -247,5 +247,5 @@
   <link name="base"/>
   <joint name="base_link-base" type="fixed">
-    <origin rpy="0 0 0" xyz="0 0 0"/>
+    <origin rpy="0 0 1.57" xyz="0 0 0"/>
     <parent link="base_link"/>
     <child link="base"/>
@@ -348,4 +348,5 @@
   <joint name="world-base_link-fixed" type="fixed">
     <parent link="world"/>
+      <origin rpy="0 0 0" xyz="0 0 0"/>
     <child link="base_link"/>
   </joint>

File: pickuppoint/urdf/pickuppoint.xacro (robot description, xacro)
@@ -4,8 +4,8 @@
     <xacro:include filename="$(find abb_resources)/urdf/common_materials.xacro" />
     <link name='world'/>
-    <gazebo reference="base_link">
+    <gazebo reference="pickuppoint">
         <material>Gazebo/Yellow</material>
     </gazebo>
-    <link name='base_link'>
+    <link name='pickuppoint'>
         <inertial>
             <mass value="100" />
@@ -181,38 +181,38 @@
         </collision>
     </link>
-    <joint name="base_link_JOINT_1" type="prismatic">
+    <joint name="pickuppoint_JOINT_1" type="prismatic">
         <origin rpy="0 0 1.57" xyz="-0.025 0 0" />
-        <parent link="base_link" />
+        <parent link="pickuppoint" />
         <child link="slider" />
         <limit effort="310" lower="0" upper="0.23" velocity="0.1" />
     </joint>
-    <joint name="world_base" type="fixed">
+    <joint name="world_pickuppoint" type="fixed">
+        <origin rpy="0 0 0" xyz="0.4 0 0" />
+        <parent link="world" />
+        <child link="pickuppoint" />
+    </joint>
+    <joint name="pickuppoint_slope" type="fixed">
         <origin rpy="0 0 0" xyz="0 0 0" />
-        <parent link="world" />
-        <child link="base_link" />
-    </joint>
-    <joint name="base_slope" type="fixed">
+        <parent link="pickuppoint" />
+        <child link="slope" />
+    </joint>
+    <joint name="pickuppoint_plateau" type="fixed">
         <origin rpy="0 0 0" xyz="0 0 0" />
-        <parent link="base_link" />
-        <child link="slope" />
-    </joint>
-    <joint name="base_plateau" type="fixed">
-        <origin rpy="0 0 0" xyz="0 0 0" />
-        <parent link="base_link" />
+        <parent link="pickuppoint" />
         <child link="plateau" />
     </joint>
-    <joint name="base_front_blocker" type="fixed">
+    <joint name="pickuppoint_front_blocker" type="fixed">
         <origin rpy="0 0 0" xyz="-0.025 0 0" />
-        <parent link="base_link" />
+        <parent link="pickuppoint" />
         <child link="front_blocker" />
     </joint>
-    <joint name="base_right_bottom_blocker" type="fixed">
+    <joint name="pickuppoint_right_bottom_blocker" type="fixed">
         <origin rpy="0 0 0" xyz="-0.025 0 0" />
-        <parent link="base_link" />
+        <parent link="pickuppoint" />
         <child link="right_bottom_blocker" />
     </joint>
-    <joint name="base_left_bottom_blocker" type="fixed">
+    <joint name="pickuppoint_left_bottom_blocker" type="fixed">
         <origin rpy="0 0 0" xyz="-0.025 0 0" />
-        <parent link="base_link" />
+        <parent link="pickuppoint" />
         <child link="left_bottom_blocker" />
     </joint>
