Commit message: Implemented substate Implemented ability to pickup puzzle peice

File: abb_irb120_gazebo/urdf/irb120_3_58.xacro (robot description, xacro)
@@ -348,5 +348,5 @@
   <joint name="world-base_link-fixed" type="fixed">
     <parent link="world"/>
-      <origin rpy="0 0 0" xyz="0 0 0"/>
+    <origin rpy="0 0 0" xyz="0 0 0"/>
     <child link="base_link"/>
   </joint>
@@ -393,5 +393,5 @@
       </material>
     </visual>
-    <collision>
+    <!-- <collision>
       <origin rpy="1.57079632679 0  -1.57079632679" xyz="0 0 0"/>
       <geometry>
@@ -401,5 +401,5 @@
         <color rgba="1 1 0 1"/>
       </material>
-    </collision>
+    </collision> -->
   </link>
   <link name="gripper2">
@@ -418,5 +418,5 @@
       </material>
     </visual>
-    <collision>
+    <!-- <collision>
       <origin rpy="1.57079632679 0  -1.57079632679" xyz="0 0 0"/>
       <geometry>
@@ -426,5 +426,5 @@
         <color rgba="1 1 0 1"/>
       </material>
-    </collision>
+    </collision> -->
   </link>
   <link name="gripper3">
@@ -443,5 +443,5 @@
       </material>
     </visual>
-    <collision>
+    <!-- <collision>
       <origin rpy="1.57079632679 0  -1.57079632679" xyz="0 0 0"/>
       <geometry>
@@ -451,5 +451,5 @@
         <color rgba="1 1 0 1"/>
       </material>
-    </collision>
+    </collision> -->
   </link>
   <link name="eef">
@@ -468,5 +468,5 @@
     <parent link="head"/>
     <child link="gripper1"/>
-    <limit effort="310" lower="0" upper="0.005" velocity="0.1"/>
+    <limit effort="5" lower="0" upper="0.0035" velocity="0.01"/>
   </joint>
   <joint name="joint_8" type="prismatic">
@@ -474,5 +474,5 @@
     <parent link="head"/>
     <child link="gripper2"/>
-    <limit effort="310" lower="0" upper="0.005" velocity="0.1"/>
+    <limit effort="5" lower="0" upper="0.0035" velocity="0.01"/>
     <mimic joint="joint_7"/>
   </joint>
@@ -481,5 +481,5 @@
     <parent link="head"/>
     <child link="gripper3"/>
-    <limit effort="310" lower="0" upper="0.005" velocity="0.1"/>
+    <limit effort="5" lower="0" upper="0.0035" velocity="0.01"/>
     <mimic joint="joint_7"/>
   </joint>
@@ -537,4 +537,31 @@
     <material>Gazebo/White</material>
     <turnGravityOff>true</turnGravityOff>
+  </gazebo>
+  <gazebo reference="joint_1">
+    <implicitSpringDamper>1</implicitSpringDamper>
+  </gazebo>
+  <gazebo reference="joint_2">
+    <implicitSpringDamper>1</implicitSpringDamper>
+  </gazebo>
+  <gazebo reference="joint_3">
+    <implicitSpringDamper>1</implicitSpringDamper>
+  </gazebo>
+  <gazebo reference="joint_4">
+    <implicitSpringDamper>1</implicitSpringDamper>
+  </gazebo>
+  <gazebo reference="joint_5">
+    <implicitSpringDamper>1</implicitSpringDamper>
+  </gazebo>
+  <gazebo reference="joint_6">
+    <implicitSpringDamper>1</implicitSpringDamper>
+  </gazebo>
+  <gazebo reference="joint_7">
+    <implicitSpringDamper>1</implicitSpringDamper>
+  </gazebo>
+  <gazebo reference="joint_8">
+    <implicitSpringDamper>1</implicitSpringDamper>
+  </gazebo>
+  <gazebo reference="joint_9">
+    <implicitSpringDamper>1</implicitSpringDamper>
   </gazebo>
   <!-- ros_control plugin -->

File: pickuppoint/urdf/pickuppoint.xacro (robot description, xacro)
@@ -33,5 +33,5 @@
     <link name='slider'>
         <inertial>
-            <mass value="5"/>
+            <mass value="0.1"/>
             <origin rpy="0 0 -1.57" xyz="0 0 0" />
             <inertia ixx="0.001" ixy="0" ixz="0" iyy="0.001" iyz="0" izz="0.001" />
@@ -40,5 +40,5 @@
             <origin rpy="0 0 -1.57" xyz="-0.39 0.02 0.28" />
             <geometry>
-                <box size="0.4 0.1 0.02"/>
+                <box size="0.4 0.1 0.03"/>
             </geometry>
             <material name="Cyan">
@@ -49,5 +49,5 @@
             <origin rpy="0 0 -1.57" xyz="-0.39 0.02 0.28" />
             <geometry>
-                <box size="0.4 0.1 0.02"/>
+                <box size="0.4 0.1 0.03"/>
             </geometry>
             <material name="Cyan">
@@ -113,16 +113,16 @@
         </inertial>
         <visual>
-            <origin rpy="0 0 0" xyz="0.02 -0.1 0.345" />
-            <geometry>
-                <box size="0.3 0.03 0.1"/>
-            </geometry>
-            <material name="Green">
-                <color rgba="0 1.0 0 1.0"/>
-            </material>
-        </visual>
-        <collision>
-            <origin rpy="0 0 0" xyz="0.02 -0.1 0.345" />
-            <geometry>
-                <box size="0.3 0.03 0.1"/>
+            <origin rpy="0 0 0" xyz="0.02 -0.1 0.355" />
+            <geometry>
+                <box size="0.3 0.03 0.08"/>
+            </geometry>
+            <material name="Green">
+                <color rgba="0 1.0 0 1.0"/>
+            </material>
+        </visual>
+        <collision>
+            <origin rpy="0 0 0" xyz="0.02 -0.1 0.355" />
+            <geometry>
+                <box size="0.3 0.03 0.08"/>
             </geometry>
             <material name="Green">

Commit message: Implemented pickup circle Implemented ability to rotate robotarm Implemented ability to rotate circle

File: abb_irb120_gazebo/urdf/irb120_3_58.xacro (robot description, xacro)
@@ -355,5 +355,5 @@
   <link name="head">
     <inertial>
-      <mass value="1"/>
+      <mass value="1000000"/>
       <origin rpy="0 0 -1.57079632679" xyz="0 0 0"/>
       <inertia ixx="0.001" ixy="0" ixz="0" iyy="0.001" iyz="0" izz="0.001"/>
@@ -380,5 +380,5 @@
   <link name="gripper1">
     <inertial>
-      <mass value="1"/>
+      <mass value="0.1"/>
       <origin rpy="1.57079632679 0  -1.57079632679" xyz="0 0 0"/>
       <inertia ixx="0.001" ixy="0" ixz="0" iyy="0.001" iyz="0" izz="0.001"/>
@@ -405,5 +405,5 @@
   <link name="gripper2">
     <inertial>
-      <mass value="1"/>
+      <mass value="0.1"/>
       <origin rpy="1.57079632679 0  -1.57079632679" xyz="0 0 0"/>
       <inertia ixx="0.001" ixy="0" ixz="0" iyy="0.001" iyz="0" izz="0.001"/>
@@ -430,5 +430,5 @@
   <link name="gripper3">
     <inertial>
-      <mass value="1"/>
+      <mass value="0.1"/>
       <origin rpy="1.57079632679 0  -1.57079632679" xyz="0 0 0"/>
       <inertia ixx="0.001" ixy="0" ixz="0" iyy="0.001" iyz="0" izz="0.001"/>
@@ -538,5 +538,5 @@
     <turnGravityOff>true</turnGravityOff>
   </gazebo>
-  <gazebo reference="joint_1">
+  <!-- <gazebo reference="joint_1">
     <implicitSpringDamper>1</implicitSpringDamper>
   </gazebo>
@@ -564,5 +564,5 @@
   <gazebo reference="joint_9">
     <implicitSpringDamper>1</implicitSpringDamper>
-  </gazebo>
+  </gazebo> -->
   <!-- ros_control plugin -->
   <joint name="joint_10" type="fixed">

Commit message: Robot can now rotate a picked up piece Robot can now drop the piece once it is correctly rotated

File: abb_irb120_gazebo/urdf/irb120_3_58.xacro (robot description, xacro)
@@ -310,5 +310,5 @@
   <gazebo reference="base_link">
     <material>Gazebo/Orange</material>
-    <turnGravityOff>true</turnGravityOff>
+    <turnGravityOff>false</turnGravityOff>
   </gazebo>
   <gazebo reference="link_1">
@@ -355,5 +355,5 @@
   <link name="head">
     <inertial>
-      <mass value="1000000"/>
+      <mass value="1"/>
       <origin rpy="0 0 -1.57079632679" xyz="0 0 0"/>
       <inertia ixx="0.001" ixy="0" ixz="0" iyy="0.001" iyz="0" izz="0.001"/>
@@ -369,4 +369,5 @@
     </visual>
     <collision>
+      <collide_bitmask>0x01</collide_bitmask>
       <origin rpy="0 0 -1.57079632679" xyz="0 0 0"/>
       <geometry>
@@ -380,5 +381,5 @@
   <link name="gripper1">
     <inertial>
-      <mass value="0.1"/>
+      <mass value="10000000000"/>
       <origin rpy="1.57079632679 0  -1.57079632679" xyz="0 0 0"/>
       <inertia ixx="0.001" ixy="0" ixz="0" iyy="0.001" iyz="0" izz="0.001"/>
@@ -393,17 +394,8 @@
       </material>
     </visual>
-    <!-- <collision>
-      <origin rpy="1.57079632679 0  -1.57079632679" xyz="0 0 0"/>
-      <geometry>
-        <mesh filename="package://schunk_mpz45/stl/SchunkSingleGripper3.stl"/>
-      </geometry>
-      <material name="">
-        <color rgba="1 1 0 1"/>
-      </material>
-    </collision> -->
   </link>
   <link name="gripper2">
     <inertial>
-      <mass value="0.1"/>
+      <mass value="10000000000"/>
       <origin rpy="1.57079632679 0  -1.57079632679" xyz="0 0 0"/>
       <inertia ixx="0.001" ixy="0" ixz="0" iyy="0.001" iyz="0" izz="0.001"/>
@@ -418,17 +410,8 @@
       </material>
     </visual>
-    <!-- <collision>
-      <origin rpy="1.57079632679 0  -1.57079632679" xyz="0 0 0"/>
-      <geometry>
-        <mesh filename="package://schunk_mpz45/stl/SchunkSingleGripper3.stl"/>
-      </geometry>
-      <material name="">
-        <color rgba="1 1 0 1"/>
-      </material>
-    </collision> -->
   </link>
   <link name="gripper3">
     <inertial>
-      <mass value="0.1"/>
+      <mass value="10000000000"/>
       <origin rpy="1.57079632679 0  -1.57079632679" xyz="0 0 0"/>
       <inertia ixx="0.001" ixy="0" ixz="0" iyy="0.001" iyz="0" izz="0.001"/>
@@ -443,13 +426,4 @@
       </material>
     </visual>
-    <!-- <collision>
-      <origin rpy="1.57079632679 0  -1.57079632679" xyz="0 0 0"/>
-      <geometry>
-        <mesh filename="package://schunk_mpz45/stl/SchunkSingleGripper3.stl"/>
-      </geometry>
-      <material name="">
-        <color rgba="1 1 0 1"/>
-      </material>
-    </collision> -->
   </link>
   <link name="eef">

File: pickuppoint/urdf/pickuppoint.xacro (robot description, xacro)
@@ -35,5 +35,5 @@
             <mass value="0.1"/>
             <origin rpy="0 0 -1.57" xyz="0 0 0" />
-            <inertia ixx="0.001" ixy="0" ixz="0" iyy="0.001" iyz="0" izz="0.001" />
+            <inertia ixx="1.0" ixy="0.0" ixz="0.0" iyy="1.0" iyz="0.0" izz="1.0" />
         </inertial>
         <visual name='visual'>
@@ -185,5 +185,5 @@
         <parent link="pickuppoint" />
         <child link="slider" />
-        <limit effort="310" lower="0" upper="0.23" velocity="0.1" />
+        <limit effort="0" lower="0" upper="0.23" velocity="0" />
     </joint>
     <joint name="world_pickuppoint" type="fixed">

Commit message: Correctly added Square positions Major bugfix for moving robot using the cartesianpath

File: abb_irb120_gazebo/urdf/irb120_3_58.xacro (robot description, xacro)
@@ -196,5 +196,5 @@
     <limit effort="0" lower="-2.87979" upper="2.87979" velocity="4.36332"/>
     <axis xyz="0 0 1"/>
-    <dynamics damping="0.0" friction="0.0"/>
+    <dynamics damping="0.2" friction="0.0"/>
   </joint>
   <joint name="joint_2" type="revolute">
@@ -204,5 +204,5 @@
     <limit effort="0" lower="-1.91986" upper="1.91986" velocity="4.36332"/>
     <axis xyz="0 1 0"/>
-    <dynamics damping="0.0" friction="0.0"/>
+    <dynamics damping="0.2" friction="0.0"/>
   </joint>
   <joint name="joint_3" type="revolute">
@@ -212,5 +212,5 @@
     <limit effort="0" lower="-1.91986" upper="1.22173" velocity="4.36332"/>
     <axis xyz="0 1 0"/>
-    <dynamics damping="0.0" friction="0.0"/>
+    <dynamics damping="0.2" friction="0.0"/>
   </joint>
   <joint name="joint_4" type="revolute">
@@ -220,5 +220,5 @@
     <limit effort="0" lower="-2.79253" upper="2.79253" velocity="5.58505"/>
     <axis xyz="1 0 0"/>
-    <dynamics damping="0.0" friction="0.0"/>
+    <dynamics damping="0.2" friction="0.0"/>
   </joint>
   <joint name="joint_5" type="revolute">
@@ -228,5 +228,5 @@
     <limit effort="0" lower="-2.094395" upper="2.094395" velocity="5.58505"/>
     <axis xyz="0 1 0"/>
-    <dynamics damping="0.0" friction="0.0"/>
+    <dynamics damping="0.2" friction="0.0"/>
   </joint>
   <joint name="joint_6" type="revolute">
@@ -236,5 +236,5 @@
     <limit effort="0" lower="-6.98132" upper="6.98132" velocity="7.33038"/>
     <axis xyz="1 0 0"/>
-    <dynamics damping="0.0" friction="0.0"/>
+    <dynamics damping="0.2" friction="0.0"/>
   </joint>
   <joint name="joint6-tool0" type="fixed">

Commit message: Square can now be pickedup and placed correctly

File: abb_irb120_gazebo/urdf/irb120_3_58.xacro (robot description, xacro)
@@ -196,5 +196,5 @@
     <limit effort="0" lower="-2.87979" upper="2.87979" velocity="4.36332"/>
     <axis xyz="0 0 1"/>
-    <dynamics damping="0.2" friction="0.0"/>
+    <dynamics damping="0.4" friction="0.0"/>
   </joint>
   <joint name="joint_2" type="revolute">
@@ -204,5 +204,5 @@
     <limit effort="0" lower="-1.91986" upper="1.91986" velocity="4.36332"/>
     <axis xyz="0 1 0"/>
-    <dynamics damping="0.2" friction="0.0"/>
+    <dynamics damping="0.4" friction="0.0"/>
   </joint>
   <joint name="joint_3" type="revolute">
@@ -212,5 +212,5 @@
     <limit effort="0" lower="-1.91986" upper="1.22173" velocity="4.36332"/>
     <axis xyz="0 1 0"/>
-    <dynamics damping="0.2" friction="0.0"/>
+    <dynamics damping="0.4" friction="0.0"/>
   </joint>
   <joint name="joint_4" type="revolute">
@@ -220,5 +220,5 @@
     <limit effort="0" lower="-2.79253" upper="2.79253" velocity="5.58505"/>
     <axis xyz="1 0 0"/>
-    <dynamics damping="0.2" friction="0.0"/>
+    <dynamics damping="0.4" friction="0.0"/>
   </joint>
   <joint name="joint_5" type="revolute">
@@ -228,5 +228,5 @@
     <limit effort="0" lower="-2.094395" upper="2.094395" velocity="5.58505"/>
     <axis xyz="0 1 0"/>
-    <dynamics damping="0.2" friction="0.0"/>
+    <dynamics damping="0.4" friction="0.0"/>
   </joint>
   <joint name="joint_6" type="revolute">
@@ -236,5 +236,5 @@
     <limit effort="0" lower="-6.98132" upper="6.98132" velocity="7.33038"/>
     <axis xyz="1 0 0"/>
-    <dynamics damping="0.2" friction="0.0"/>
+    <dynamics damping="0.4" friction="0.0"/>
   </joint>
   <joint name="joint6-tool0" type="fixed">

Commit message: Rectangles can now be correctly placed and rotated

File: abb_irb120_gazebo/urdf/irb120_3_58.xacro (robot description, xacro)
@@ -196,5 +196,5 @@
     <limit effort="0" lower="-2.87979" upper="2.87979" velocity="4.36332"/>
     <axis xyz="0 0 1"/>
-    <dynamics damping="0.4" friction="0.0"/>
+    <dynamics damping="0.4" friction="100.0"/>
   </joint>
   <joint name="joint_2" type="revolute">
@@ -204,5 +204,5 @@
     <limit effort="0" lower="-1.91986" upper="1.91986" velocity="4.36332"/>
     <axis xyz="0 1 0"/>
-    <dynamics damping="0.4" friction="0.0"/>
+    <dynamics damping="0.4" friction="100.0"/>
   </joint>
   <joint name="joint_3" type="revolute">
@@ -212,5 +212,5 @@
     <limit effort="0" lower="-1.91986" upper="1.22173" velocity="4.36332"/>
     <axis xyz="0 1 0"/>
-    <dynamics damping="0.4" friction="0.0"/>
+    <dynamics damping="0.4" friction="100.0"/>
   </joint>
   <joint name="joint_4" type="revolute">
@@ -220,5 +220,5 @@
     <limit effort="0" lower="-2.79253" upper="2.79253" velocity="5.58505"/>
     <axis xyz="1 0 0"/>
-    <dynamics damping="0.4" friction="0.0"/>
+    <dynamics damping="0.4" friction="100.0"/>
   </joint>
   <joint name="joint_5" type="revolute">
@@ -228,5 +228,5 @@
     <limit effort="0" lower="-2.094395" upper="2.094395" velocity="5.58505"/>
     <axis xyz="0 1 0"/>
-    <dynamics damping="0.4" friction="0.0"/>
+    <dynamics damping="0.4" friction="100.0"/>
   </joint>
   <joint name="joint_6" type="revolute">
@@ -236,5 +236,5 @@
     <limit effort="0" lower="-6.98132" upper="6.98132" velocity="7.33038"/>
     <axis xyz="1 0 0"/>
-    <dynamics damping="0.4" friction="0.0"/>
+    <dynamics damping="0.4" friction="100.0"/>
   </joint>
   <joint name="joint6-tool0" type="fixed">

Commit message: Fixed bug which caused grippers not to move

File: abb_irb120_gazebo/urdf/irb120_3_58.xacro (robot description, xacro)
@@ -310,5 +310,5 @@
   <gazebo reference="base_link">
     <material>Gazebo/Orange</material>
-    <turnGravityOff>false</turnGravityOff>
+    <turnGravityOff>true</turnGravityOff>
   </gazebo>
   <gazebo reference="link_1">
@@ -355,5 +355,5 @@
   <link name="head">
     <inertial>
-      <mass value="1"/>
+      <mass value="1000000"/>
       <origin rpy="0 0 -1.57079632679" xyz="0 0 0"/>
       <inertia ixx="0.001" ixy="0" ixz="0" iyy="0.001" iyz="0" izz="0.001"/>
@@ -381,5 +381,5 @@
   <link name="gripper1">
     <inertial>
-      <mass value="10000000000"/>
+      <mass value="0.1"/>
       <origin rpy="1.57079632679 0  -1.57079632679" xyz="0 0 0"/>
       <inertia ixx="0.001" ixy="0" ixz="0" iyy="0.001" iyz="0" izz="0.001"/>
@@ -397,5 +397,5 @@
   <link name="gripper2">
     <inertial>
-      <mass value="10000000000"/>
+      <mass value="0.1"/>
       <origin rpy="1.57079632679 0  -1.57079632679" xyz="0 0 0"/>
       <inertia ixx="0.001" ixy="0" ixz="0" iyy="0.001" iyz="0" izz="0.001"/>
@@ -413,5 +413,5 @@
   <link name="gripper3">
     <inertial>
-      <mass value="10000000000"/>
+      <mass value="0.1"/>
       <origin rpy="1.57079632679 0  -1.57079632679" xyz="0 0 0"/>
       <inertia ixx="0.001" ixy="0" ixz="0" iyy="0.001" iyz="0" izz="0.001"/>

Commit message: Fixed: Difference in simulation and moveit Fixed: Placement of pieces in correct sized puzzle

File: abb_irb120_gazebo/urdf/irb120_3_58.xacro (robot description, xacro)
@@ -196,5 +196,5 @@
     <limit effort="0" lower="-2.87979" upper="2.87979" velocity="4.36332"/>
     <axis xyz="0 0 1"/>
-    <dynamics damping="0.4" friction="100.0"/>
+    <dynamics damping="0.4" friction="0.0"/>
   </joint>
   <joint name="joint_2" type="revolute">
@@ -204,5 +204,5 @@
     <limit effort="0" lower="-1.91986" upper="1.91986" velocity="4.36332"/>
     <axis xyz="0 1 0"/>
-    <dynamics damping="0.4" friction="100.0"/>
+    <dynamics damping="0.4" friction="0.0"/>
   </joint>
   <joint name="joint_3" type="revolute">
@@ -212,5 +212,5 @@
     <limit effort="0" lower="-1.91986" upper="1.22173" velocity="4.36332"/>
     <axis xyz="0 1 0"/>
-    <dynamics damping="0.4" friction="100.0"/>
+    <dynamics damping="0.4" friction="0.0"/>
   </joint>
   <joint name="joint_4" type="revolute">
@@ -220,5 +220,5 @@
     <limit effort="0" lower="-2.79253" upper="2.79253" velocity="5.58505"/>
     <axis xyz="1 0 0"/>
-    <dynamics damping="0.4" friction="100.0"/>
+    <dynamics damping="0.4" friction="0.0"/>
   </joint>
   <joint name="joint_5" type="revolute">
@@ -228,5 +228,5 @@
     <limit effort="0" lower="-2.094395" upper="2.094395" velocity="5.58505"/>
     <axis xyz="0 1 0"/>
-    <dynamics damping="0.4" friction="100.0"/>
+    <dynamics damping="0.4" friction="0.0"/>
   </joint>
   <joint name="joint_6" type="revolute">
@@ -236,5 +236,5 @@
     <limit effort="0" lower="-6.98132" upper="6.98132" velocity="7.33038"/>
     <axis xyz="1 0 0"/>
-    <dynamics damping="0.4" friction="100.0"/>
+    <dynamics damping="0.4" friction="0.0"/>
   </joint>
   <joint name="joint6-tool0" type="fixed">

File: pickuppoint/urdf/pickuppoint.xacro (robot description, xacro)
@@ -182,9 +182,7 @@
     </link>
     <joint name="pickuppoint_JOINT_1" type="prismatic">
-        <origin rpy="0 0 1.57" xyz="-0.025 0 0" />
+        <origin rpy="0 -0.00005 1.57" xyz="-0.025 0 0" />
         <parent link="pickuppoint" />
         <child link="slider" />
-        <spring_stiffness>111.1111</spring_stiffness>
-        <spring_reference>1.0</spring_reference>
         <damping>0.0</damping>
         <friction>0.0</friction>

Commit message: Robot can now Pickup all physical puzzlepieces.

File: abb_irb120_gazebo/urdf/irb120_3_58.xacro (robot description, xacro)
@@ -234,5 +234,5 @@
     <parent link="link_5"/>
     <child link="link_6"/>
-    <limit effort="0" lower="-6.98132" upper="6.98132" velocity="7.33038"/>
+    <limit effort="0" lower="-3.1415" upper="3.1415" velocity="7.33038"/>
     <axis xyz="1 0 0"/>
     <dynamics damping="0.4" friction="0.0"/>

File: abb_irb120_support/urdf/irb120_3_58.urdf (robot description, URDF)
Before this commit: robot abb_irb120_schunk_mpz45, 15 links, 14 joints
Joints:
- joint joint_6: limit lower=-6.98132 upper=6.98132 effort=0 velocity=7.33038 -> lower=-3.1415 upper=3.1415 effort=0 velocity=7.33038

Commit message: Square and rectangle can now be rotated correct.

File: abb_irb120_gazebo/urdf/irb120_3_58.xacro (robot description, xacro)
@@ -234,5 +234,5 @@
     <parent link="link_5"/>
     <child link="link_6"/>
-    <limit effort="0" lower="-3.1415" upper="3.1415" velocity="7.33038"/>
+    <limit effort="0" lower="-6.283" upper="6.283" velocity="7.33038"/>
     <axis xyz="1 0 0"/>
     <dynamics damping="0.4" friction="0.0"/>

File: abb_irb120_support/urdf/irb120_3_58.urdf (robot description, URDF)
Before this commit: robot abb_irb120_schunk_mpz45, 15 links, 14 joints
Joints:
- joint joint_6: limit lower=-3.1415 upper=3.1415 effort=0 velocity=7.33038 -> lower=-6.283 upper=6.283 effort=0 velocity=7.33038
