Commit message: Added points for pickuppoint slider

File: abb_irb120_support/urdf/irb120_3_58.urdf (robot description, URDF)
Before this commit: robot abb_irb120_3_58, 9 links, 8 joints
Links:
- added link eef; visual sphere radius=0.001
- added link gripper1, mass 1; collision mesh filename=package://schunk_mpz45/stl/SchunkSingleGripper3.stl; visual mesh filename=package://schunk_mpz45/stl/SchunkSingleGripper3.stl
- added link gripper2, mass 1; collision mesh filename=package://schunk_mpz45/stl/SchunkSingleGripper3.stl; visual mesh filename=package://schunk_mpz45/stl/SchunkSingleGripper3.stl
- added link gripper3, mass 1; collision mesh filename=package://schunk_mpz45/stl/SchunkSingleGripper3.stl; visual mesh filename=package://schunk_mpz45/stl/SchunkSingleGripper3.stl
- added link head, mass 1; collision mesh filename=package://schunk_mpz45/stl/SchunkGripperNoGripperCorrect.stl; visual mesh filename=package://schunk_mpz45/stl/SchunkGripperNoGripperCorrect.stl
- added link world
Joints:
- added joint eef-head: type fixed, parent head, child eef, origin xyz=0.05 0 0 rpy=0 0 0
- added joint joint_10: type fixed, parent tool0, child head, origin xyz=0 0 0 rpy=0 0 0
- added joint joint_7: type prismatic, parent head, child gripper1, origin xyz=0 0 0 rpy=-1.57079632679 -2.61799387799 -1.57079632679, limit lower=0 upper=0.005 effort=310 velocity=0.1
- added joint joint_8: type prismatic, parent head, child gripper2, origin xyz=0 0 0 rpy=-1.57079632679 -0.523598775598 -1.57079632679, limit lower=0 upper=0.005 effort=310 velocity=0.1, mimic joint=joint_7
- added joint joint_9: type prismatic, parent head, child gripper3, origin xyz=0 0 0 rpy=0 1.57079632679 0, limit lower=0 upper=0.005 effort=310 velocity=0.1, mimic joint=joint_7
- added joint world-base_link-fixed: type fixed, parent world, child base_link
