Commit message: Add capacitive sensors to pickuppoint Minor changes in pickuppoint to increase correctly falling of puzzlepiecse

File: pickuppoint/urdf/pickuppoint.xacro (robot description, xacro)
@@ -4,22 +4,25 @@
     <xacro:include filename="$(find abb_resources)/urdf/common_materials.xacro" />
     <link name='world'/>
+    <gazebo reference="base_link">
+        <material>Gazebo/Yellow</material>
+    </gazebo>
     <link name='base_link'>
-    <inertial>
-      <mass value="100" />
-      <inertia ixx="1.0" ixy="0.0" ixz="0.0" iyy="1.0" iyz="0.0" izz="1.0" />
-    </inertial>
-        <visual name='visual'>
-            <origin rpy="0 0 0" xyz="0.025 0.395 0" />
+        <inertial>
+            <mass value="100" />
+            <inertia ixx="1.0" ixy="0.0" ixz="0.0" iyy="1.0" iyz="0.0" izz="1.0" />
+        </inertial>
+        <visual>
+            <origin rpy="0 0 0" xyz="0.00 0.395 0" />
             <geometry>
-                <mesh filename="package://pickuppoint/stl/lowResPickupPoint.stl" />
+                <mesh filename="package://pickuppoint/stl/lowResPickupPointNoFrontWall.stl" />
             </geometry>
-            <material name="Red">
+            <material name="red">
                 <color rgba="1 0 0 1.0"/>
             </material>
         </visual>
         <collision>
-            <origin rpy="0 0 0" xyz="0.025 0.395 0" />
+            <origin rpy="0 0 0" xyz="0.0 0.395 0" />
             <geometry>
-                <mesh filename="package://pickuppoint/stl/lowResPickupPoint.stl" />
+                <mesh filename="package://pickuppoint/stl/lowResPickupPointNoFrontWall.stl" />
             </geometry>
             <material name="">
@@ -30,5 +33,5 @@
     <link name='link_1'>
         <inertial>
-            <mass value="1"/>
+            <mass value="5"/>
             <origin rpy="0 0 -1.57" xyz="0 0 0" />
             <inertia ixx="0.001" ixy="0" ixz="0" iyy="0.001" iyz="0" izz="0.001" />
@@ -60,5 +63,5 @@
         </inertial>
         <visual name='visual'>
-            <origin rpy="0 0 0" xyz="0 -0.27 0.273" />
+            <origin rpy="0 0 0" xyz="0 -0.2645 0.271" />
             <geometry>
                 <box size="0.26 0.36 0.002"/>
@@ -78,6 +81,81 @@
         </collision>
     </link>
+    <link name='link_3'>
+        <inertial>
+            <mass value="1"/>
+            <origin rpy="0 0 0" xyz="0 0 0" />
+            <inertia ixx="0.001" ixy="0" ixz="0" iyy="0.001" iyz="0" izz="0.001" />
+        </inertial>
+        <visual>
+            <origin rpy="0 0 0" xyz="0.02 -0.1 0.345" />
+            <geometry>
+                <box size="0.3 0.03 0.1"/>
+            </geometry>
+            <material name="Green">
+                <color rgba="0 1.0 0 1.0"/>
+            </material>
+        </visual>
+        <collision>
+            <origin rpy="0 0 0" xyz="0.02 -0.1 0.345" />
+            <geometry>
+                <box size="0.3 0.03 0.1"/>
+            </geometry>
+            <material name="Green">
+                <color rgba="0 1.0 0 1.0"/>
+            </material>
+        </collision>
+    </link>
+    <link name='link_4'>
+        <inertial>
+            <mass value="1"/>
+            <origin rpy="0 0 0" xyz="0 0 0" />
+            <inertia ixx="0.001" ixy="0" ixz="0" iyy="0.001" iyz="0" izz="0.001" />
+        </inertial>
+        <visual>
+            <origin rpy="-0.39 0.38 0.70" xyz="-0.10 0.245 0.1" />
+            <geometry>
+                <box size="0.34 0.035 0.035"/>
+            </geometry>
+            <material name="Green">
+                <color rgba="0 1.0 0 1.0"/>
+            </material>
+        </visual>
+        <collision>
+            <origin rpy="-0.39 0.38 0.70" xyz="-0.10 0.245 0.1" />
+            <geometry>
+                <box size="0.34 0.035 0.035"/>
+            </geometry>
+            <material name="Green">
+                <color rgba="0 1.0 0 1.0"/>
+            </material>
+        </collision>
+    </link>
+    <link name='link_5'>
+        <inertial>
+            <mass value="1"/>
+            <origin rpy="0 0 0" xyz="0 0 0" />
+            <inertia ixx="0.001" ixy="0" ixz="0" iyy="0.001" iyz="0" izz="0.001" />
+        </inertial>
+        <visual>
+            <origin rpy="-0.39 -0.38 -0.7" xyz="0.15 0.245 0.1" />
+            <geometry>
+                <box size="0.34 0.035 0.035"/>
+            </geometry>
+            <material name="Green">
+                <color rgba="0 1.0 0 1.0"/>
+            </material>
+        </visual>
+        <collision>
+            <origin rpy="-0.39 -0.38 -0.7" xyz="0.15 0.245 0.1" />
+            <geometry>
+                <box size="0.34 0.035 0.035"/>
+            </geometry>
+            <material name="Green">
+                <color rgba="0 1.0 0 1.0"/>
+            </material>
+        </collision>
+    </link>
     <joint name="base_link_JOINT_1" type="prismatic">
-        <origin rpy="0 0 1.57" xyz="0 0 0" />
+        <origin rpy="0 0 1.57" xyz="-0.025 0 0" />
         <parent link="base_link" />
         <child link="link_1" />
@@ -89,9 +167,24 @@
         <child link="base_link" />
     </joint>
-     <joint name="base_link2" type="fixed">
+    <joint name="base_link2" type="fixed">
         <origin rpy="0 0 0" xyz="0 0 0" />
         <parent link="base_link" />
         <child link="link_2" />
     </joint>
+    <joint name="base_link3" type="fixed">
+        <origin rpy="0 0 0" xyz="-0.025 0 0" />
+        <parent link="base_link" />
+        <child link="link_3" />
+    </joint>
+    <joint name="base_link4" type="fixed">
+        <origin rpy="0 0 0" xyz="-0.025 0 0" />
+        <parent link="base_link" />
+        <child link="link_4" />
+    </joint>
+    <joint name="base_link5" type="fixed">
+        <origin rpy="0 0 0" xyz="-0.025 0 0" />
+        <parent link="base_link" />
+        <child link="link_5" />
+    </joint>
     <!-- </xacro:macro> -->
 </robot>

Commit message: Puzzle with sensors implemented

File: pickuppoint/urdf/pickuppoint.xacro (robot description, xacro)
@@ -187,4 +187,3 @@
         <child link="link_5" />
     </joint>
-    <!-- </xacro:macro> -->
 </robot>

Commit message: Decreasement of pickup-stl for performance gain

File: pickuppoint/urdf/pickuppoint.xacro (robot description, xacro)
@@ -15,5 +15,5 @@
             <origin rpy="0 0 0" xyz="0.00 0.395 0" />
             <geometry>
-                <mesh filename="package://pickuppoint/stl/lowResPickupPointNoFrontWall.stl" />
+                <mesh filename="package://pickuppoint/stl/ultimateLowResPickupPoint2.0.stl" />
             </geometry>
             <material name="red">
@@ -24,5 +24,5 @@
             <origin rpy="0 0 0" xyz="0.0 0.395 0" />
             <geometry>
-                <mesh filename="package://pickuppoint/stl/lowResPickupPointNoFrontWall.stl" />
+                <mesh filename="package://pickuppoint/stl/ultimateLowResPickupPoint2.0.stl" />
             </geometry>
             <material name="">
@@ -31,5 +31,5 @@
         </collision>
     </link>
-    <link name='link_1'>
+    <link name='slider'>
         <inertial>
             <mass value="5"/>
@@ -56,5 +56,5 @@
         </collision>
     </link>
-    <link name='link_2'>
+    <link name='plateau'>
         <inertial>
             <mass value="1"/>
@@ -63,5 +63,5 @@
         </inertial>
         <visual name='visual'>
-            <origin rpy="0 0 0" xyz="0 -0.2645 0.271" />
+            <origin rpy="0 0 0" xyz="0 -0.2645 0.273" />
             <geometry>
                 <box size="0.26 0.36 0.002"/>
@@ -81,5 +81,30 @@
         </collision>
     </link>
-    <link name='link_3'>
+    <link name='slope'>
+        <inertial>
+            <mass value="1"/>
+            <origin rpy="0 0 0" xyz="0 0 0" />
+            <inertia ixx="0.001" ixy="0" ixz="0" iyy="0.001" iyz="0" izz="0.001" />
+        </inertial>
+        <visual name='visual'>
+            <origin rpy="-0.53 0 0" xyz="0 0.014 0.204" />
+            <geometry>
+                <box size="0.24 0.24 0.02"/>
+            </geometry>
+            <material name="Green">
+                <color rgba="0 1.0 0 1.0"/>
+            </material>
+        </visual>
+        <collision>
+            <origin rpy="-0.53 0 0" xyz="0 0.014 0.204" />
+            <geometry>
+                <box size="0.24 0.24 0.02"/>
+            </geometry>
+            <material name="Green">
+                <color rgba="0 1.0 0 1.0"/>
+            </material>
+        </collision>
+    </link>
+    <link name='front_blocker'>
         <inertial>
             <mass value="1"/>
@@ -106,5 +131,5 @@
         </collision>
     </link>
-    <link name='link_4'>
+    <link name='right_bottom_blocker'>
         <inertial>
             <mass value="1"/>
@@ -131,5 +156,5 @@
         </collision>
     </link>
-    <link name='link_5'>
+    <link name='left_bottom_blocker'>
         <inertial>
             <mass value="1"/>
@@ -159,5 +184,5 @@
         <origin rpy="0 0 1.57" xyz="-0.025 0 0" />
         <parent link="base_link" />
-        <child link="link_1" />
+        <child link="slider" />
         <limit effort="310" lower="0" upper="0.23" velocity="0.1" />
     </joint>
@@ -167,23 +192,28 @@
         <child link="base_link" />
     </joint>
-    <joint name="base_link2" type="fixed">
+    <joint name="base_slope" type="fixed">
         <origin rpy="0 0 0" xyz="0 0 0" />
         <parent link="base_link" />
-        <child link="link_2" />
-    </joint>
-    <joint name="base_link3" type="fixed">
+        <child link="slope" />
+    </joint>
+    <joint name="base_plateau" type="fixed">
+        <origin rpy="0 0 0" xyz="0 0 0" />
+        <parent link="base_link" />
+        <child link="plateau" />
+    </joint>
+    <joint name="base_front_blocker" type="fixed">
         <origin rpy="0 0 0" xyz="-0.025 0 0" />
         <parent link="base_link" />
-        <child link="link_3" />
-    </joint>
-    <joint name="base_link4" type="fixed">
+        <child link="front_blocker" />
+    </joint>
+    <joint name="base_right_bottom_blocker" type="fixed">
         <origin rpy="0 0 0" xyz="-0.025 0 0" />
         <parent link="base_link" />
-        <child link="link_4" />
-    </joint>
-    <joint name="base_link5" type="fixed">
+        <child link="right_bottom_blocker" />
+    </joint>
+    <joint name="base_left_bottom_blocker" type="fixed">
         <origin rpy="0 0 0" xyz="-0.025 0 0" />
         <parent link="base_link" />
-        <child link="link_5" />
+        <child link="left_bottom_blocker" />
     </joint>
 </robot>

Commit message: Implemented move and movestraight action

File: pickuppoint/urdf/pickuppoint.xacro (robot description, xacro)
@@ -15,5 +15,5 @@
             <origin rpy="0 0 0" xyz="0.00 0.395 0" />
             <geometry>
-                <mesh filename="package://pickuppoint/stl/PickupPoint.stl" />
+                <mesh filename="package://pickuppoint/stl/ultimateLowResPickupPoint2.0.stl" />
             </geometry>
             <material name="red">

Commit message: Added the simulator for the slider

File: pickuppoint/urdf/pickuppoint.xacro (robot description, xacro)
@@ -33,5 +33,5 @@
     <link name='slider'>
         <inertial>
-            <mass value="0.1"/>
+            <mass value="1.0"/>
             <origin rpy="0 0 -1.57" xyz="0 0 0" />
             <inertia ixx="1.0" ixy="0.0" ixz="0.0" iyy="1.0" iyz="0.0" izz="1.0" />
